File: SEGmeterShield15.sch (EAGLE design)
At the start: 68 parts, among them IC1 MCP1541, IC2 MCP3208, J1 Sensor 5V, J10 3.5mm, J11 Star ground, J12 3.5mm, J13 Arduino-compatible headers, J14 3.5mm, J15 3.5mm, J2 3.5mm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

Commit message: foo
Other:
- note added: "Smart Energy Groups SEGShield v1.5"
- note added: "V1.5 (03-07-2012)"
- note removed: "Smart Energy Groups SEGmeter v2.5"
- note removed: "V0.5 (03-07-2012)"
Changed lines of the file:
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@@
 <wire x1="281.94" y1="17.78" x2="281.94" y2="12.7" width="0.3048" layer="94"/>
 <wire x1="312.166" y1="17.78" x2="312.166" y2="12.7" width="0.3048" layer="94"/>
-<text x="259.08" y="20.32" size="3.048" layer="94">Smart Energy Groups SEGmeter v2.5</text>
-<text x="284.48" y="14.478" size="1.778" layer="94">V0.5 (03-07-2012)</text>
+<text x="259.08" y="20.32" size="3.048" layer="94">Smart Energy Groups SEGShield v1.5</text>
+<text x="284.48" y="14.478" size="1.778" layer="94">V1.5 (03-07-2012)</text>
 <text x="259.08" y="14.478" size="1.778" layer="94">foo</text>
 <text x="258.826" y="9.398" size="1.778" layer="94">(C)2012 Luke Weston</text>
@@
 <wire x1="71.12" y1="17.78" x2="71.12" y2="12.7" width="0.3048" layer="94"/>
 <wire x1="101.346" y1="17.78" x2="101.346" y2="12.7" width="0.3048" layer="94"/>
-<text x="48.26" y="20.32" size="3.048" layer="94">Smart Energy Groups SEGmeter v2.5</text>
-<text x="73.66" y="14.478" size="1.778" layer="94">V0.5 (03-07-2012)</text>
+<text x="48.26" y="20.32" size="3.048" layer="94">Smart Energy Groups SEGShield v1.5</text>
+<text x="73.66" y="14.478" size="1.778" layer="94">V1.5 (03-07-2012)</text>
 <text x="48.26" y="14.478" size="1.778" layer="94">foo</text>
 <text x="48.006" y="9.398" size="1.778" layer="94">(C)2012 Luke Weston</text>
