File: SEGmeterShield15.brd (EAGLE design)
At the start: 104.1 x 76.8 mm, 69 parts, among them IC1 MCP1541, IC2 MCP3208, J1 Sensor 5V, J10 3.5mm, J11 Star ground, J12 3.5mm, J13 Arduino-compatible headers, J14 3.5mm, J15 3.5mm, J2 3.5mm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

Commit message: foo
Parts:
- moved J11 1.31 mm to (42.5, 46.7)
Changed lines of the file:
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@@
 <text x="77.47" y="30.48" size="0.8128" layer="21" ratio="15">Released under the CERN OH License:</text>
 <text x="77.47" y="29.21" size="0.8128" layer="21" ratio="15">http://ohwr.org/cernohl</text>
-<text x="36.83" y="46.355" size="0.8128" layer="21" ratio="15">GND/</text>
-<text x="36.83" y="45.085" size="0.8128" layer="21" ratio="15">AGND</text>
+<text x="38.4175" y="46.6725" size="0.8128" layer="21" ratio="15">GND/</text>
+<text x="38.4175" y="45.56125" size="0.8128" layer="21" ratio="15">AGND</text>
 <text x="73.66" y="34.925" size="0.8128" layer="21" ratio="15">Compatible with most Arduino-like devices</text>
 <text x="33.655" y="66.19875" size="0.8128" layer="21" ratio="15">A5</text>
@@
 <text x="30.7975" y="47.14875" size="0.8128" layer="21" ratio="15">GND</text>
 <wire x1="7.62" y1="50.8" x2="7.62" y2="50.165" width="0.4064" layer="21"/>
+<dimension x1="0" y1="73.025" x2="104.14" y2="73.025" x3="52.07" y3="78.74" layer="48"/>
 </plain>
 <attributes>
@@
 <attribute name="VALUE" x="59.309" y="30.0355" size="0.762" layer="27" ratio="12"/>
 </element>
-<element name="J11" library="freetronics-luke" package="SJ" value="Star ground" x="41.275" y="46.355" smashed="yes" rot="R270"/>
+<element name="J11" library="freetronics-luke" package="SJ" value="Star ground" x="42.545" y="46.6725" smashed="yes" rot="R270"/>
 <element name="IC1" library="freetronics-luke" package="TO92-STRAIGHT" value="MCP1541" x="43.259375" y="41.91" smashed="yes" rot="R90">
 <attribute name="VALUE" x="40.9575" y="38.179375" size="0.762" layer="27" ratio="12"/>
